Commit message: Add companion depth camera sensor macro

File: orange_ros2/orange_description/xacro/sensors/rgb_camera.xacro (robot description, xacro)
@@ -50,3 +50,34 @@
     </gazebo>
   </xacro:macro>
+  <!--
+    Depth stream companion for an existing camera link. Keeping the depth
+    sensor separate preserves the already-validated RGB topic contract while
+    allowing the two simulated streams to share one physical pose and optical
+    frame, similar to a RealSense-style RGB-D device.
+  -->
+  <xacro:macro name="sensor_depth_camera"
+               params="name parent image_topic camera_info_topic frame_id width height update_rate hfov near_clip far_clip">
+    <gazebo reference="${parent}">
+      <sensor type="depth_camera" name="${name}">
+        <always_on>true</always_on>
+        <visualize>true</visualize>
+        <update_rate>${update_rate}</update_rate>
+        <topic>${image_topic}</topic>
+        <gz_frame_id>${frame_id}</gz_frame_id>
+        <camera name="${name}">
+          <camera_info_topic>${camera_info_topic}</camera_info_topic>
+          <horizontal_fov>${hfov}</horizontal_fov>
+          <image>
+            <width>${width}</width>
+            <height>${height}</height>
+            <format>R_FLOAT32</format>
+          </image>
+          <clip>
+            <near>${near_clip}</near>
+            <far>${far_clip}</far>
+          </clip>
+        </camera>
+      </sensor>
+    </gazebo>
+  </xacro:macro>
 </robot>
