Commit message: Resize simulation robot footprint for IGVC scale

File: orange_ros2/orange_description/xacro/orange_robot_simulation.xacro (robot description, xacro)
@@ -1,4 +1,11 @@
 <?xml version="1.0"?>
 <robot xmlns:xacro="http://www.ros.org/wiki/xacro" name="orange_robot">
+  <!-- Simulation footprint parameters. Replace with measured robot dimensions later. -->
+  <xacro:property name="base_length" value="1.00"/>
+  <xacro:property name="base_width" value="0.70"/>
+  <xacro:property name="wheel_separation" value="0.65"/>
+  <xacro:property name="wheel_radius" value="0.10"/>
+  <xacro:property name="caster_x" value="0.44"/>
+  <xacro:property name="caster_y" value="0.27"/>
   <!-- 1. 시뮬레이션 플러그인 & 센서 기능 -->
   <xacro:include filename="$(find orange_description)/xacro/orange_robot_simulation.gazebo"/>
@@ -23,15 +30,16 @@
     <visual>
       <origin xyz="0 0 0.15" rpy="0 0 0"/>
-      <geometry><box size="0.8 0.5 0.3"/></geometry>
+      <geometry><box size="${base_length} ${base_width} 0.3"/></geometry>
       <material name="yellow"/>
     </visual>
     <collision>
       <origin xyz="0 0 0.15" rpy="0 0 0"/>
-      <geometry><box size="0.8 0.5 0.3"/></geometry>
+      <geometry><box size="${base_length} ${base_width} 0.3"/></geometry>
     </collision>
     <inertial>
       <mass value="27.1"/>
       <origin xyz="0 0 0.15" rpy="0 0 0"/>
-      <inertia ixx="0.7803" ixy="0.0" ixz="0.0" iyy="0.8839" iyz="0.0" izz="1.2577"/>
+      <!-- Uniform-box approximation for the 1.00 x 0.70 x 0.30 m baseline body. -->
+      <inertia ixx="1.3098" ixy="0.0" ixz="0.0" iyy="2.4616" iyz="0.0" izz="3.3649"/>
     </inertial>
   </link>
@@ -47,5 +55,5 @@
   <link name="top_cover">
     <visual>
-      <geometry><box size="0.8 0.5 0.02"/></geometry>
+      <geometry><box size="${base_length} ${base_width} 0.02"/></geometry>
       <material name="grey"/>
     </visual>
@@ -90,32 +98,32 @@
   <joint name="left_wheel_hinge" type="continuous">
     <parent link="base_link"/><child link="left_wheel"/>
-    <origin xyz="0 0.28 0" rpy="-1.5707 0 0"/>
+    <origin xyz="0 ${wheel_separation / 2.0} 0" rpy="-1.5707 0 0"/>
     <axis xyz="0 0 1"/>
     <limit effort="100" velocity="100.0"/>
   </joint>
   <link name="left_wheel">
-    <visual><geometry><cylinder radius="0.1" length="0.05"/></geometry><material name="black"/></visual>
-    <collision><geometry><cylinder radius="0.1" length="0.05"/></geometry></collision>
+    <visual><geometry><cylinder radius="${wheel_radius}" length="0.05"/></geometry><material name="black"/></visual>
+    <collision><geometry><cylinder radius="${wheel_radius}" length="0.05"/></geometry></collision>
     <inertial><mass value="3.4"/><origin xyz="0 0 0"/><inertia ixx="0.009" ixy="0.0" ixz="0.0" iyy="0.009" iyz="0.0" izz="0.017"/></inertial>
   </link>
   <joint name="right_wheel_hinge" type="continuous">
     <parent link="base_link"/><child link="right_wheel"/>
-    <origin xyz="0 -0.28 0" rpy="-1.5707 0 0"/>
+    <origin xyz="0 ${-wheel_separation / 2.0} 0" rpy="-1.5707 0 0"/>
     <axis xyz="0 0 1"/>
     <limit effort="100" velocity="100.0"/>
   </joint>
   <link name="right_wheel">
-    <visual><geometry><cylinder radius="0.1" length="0.05"/></geometry><material name="black"/></visual>
-    <collision><geometry><cylinder radius="0.1" length="0.05"/></geometry></collision>
+    <visual><geometry><cylinder radius="${wheel_radius}" length="0.05"/></geometry><material name="black"/></visual>
+    <collision><geometry><cylinder radius="${wheel_radius}" length="0.05"/></geometry></collision>
     <inertial><mass value="3.4"/><origin xyz="0 0 0"/><inertia ixx="0.009" ixy="0.0" ixz="0.0" iyy="0.009" iyz="0.0" izz="0.017"/></inertial>
   </link>
   <!-- 8. 보조 바퀴 (캐스터 4개) -->
-  <joint name="fl_caster_joint" type="fixed"><parent link="base_link"/><child link="fl_caster"/><origin xyz="0.35 0.2 -0.05" rpy="0 0 0"/></joint>
+  <joint name="fl_caster_joint" type="fixed"><parent link="base_link"/><child link="fl_caster"/><origin xyz="${caster_x} ${caster_y} -0.05" rpy="0 0 0"/></joint>
   <link name="fl_caster"><visual><geometry><sphere radius="0.05"/></geometry><material name="black"/></visual><collision><geometry><sphere radius="0.05"/></geometry></collision></link>
-  <joint name="fr_caster_joint" type="fixed"><parent link="base_link"/><child link="fr_caster"/><origin xyz="0.35 -0.2 -0.05" rpy="0 0 0"/></joint>
+  <joint name="fr_caster_joint" type="fixed"><parent link="base_link"/><child link="fr_caster"/><origin xyz="${caster_x} ${-caster_y} -0.05" rpy="0 0 0"/></joint>
   <link name="fr_caster"><visual><geometry><sphere radius="0.05"/></geometry><material name="black"/></visual><collision><geometry><sphere radius="0.05"/></geometry></collision></link>
-  <joint name="rl_caster_joint" type="fixed"><parent link="base_link"/><child link="rl_caster"/><origin xyz="-0.35 0.2 -0.05" rpy="0 0 0"/></joint>
+  <joint name="rl_caster_joint" type="fixed"><parent link="base_link"/><child link="rl_caster"/><origin xyz="${-caster_x} ${caster_y} -0.05" rpy="0 0 0"/></joint>
   <link name="rl_caster"><visual><geometry><sphere radius="0.05"/></geometry><material name="black"/></visual><collision><geometry><sphere radius="0.05"/></geometry></collision></link>
-  <joint name="rr_caster_joint" type="fixed"><parent link="base_link"/><child link="rr_caster"/><origin xyz="-0.35 -0.2 -0.05" rpy="0 0 0"/></joint>
+  <joint name="rr_caster_joint" type="fixed"><parent link="base_link"/><child link="rr_caster"/><origin xyz="${-caster_x} ${-caster_y} -0.05" rpy="0 0 0"/></joint>
   <link name="rr_caster"><visual><geometry><sphere radius="0.05"/></geometry><material name="black"/></visual><collision><geometry><sphere radius="0.05"/></geometry></collision></link>
 </robot>

Commit message: Add front competition-compatible RGB camera to simulation

File: orange_ros2/orange_description/xacro/orange_robot_simulation.xacro (robot description, xacro)
@@ -13,4 +13,5 @@
   <xacro:include filename="$(find orange_description)/xacro/sensors/livox_simulation.xacro"/>
   <xacro:include filename="$(find orange_description)/xacro/sensors/imu.xacro"/>
+  <xacro:include filename="$(find orange_description)/xacro/sensors/rgb_camera.xacro"/>
   <!-- 색상 물감 준비 -->
   <material name="yellow"><color rgba="0.9 0.8 0.0 1.0"/></material>
@@ -74,5 +75,5 @@
     <visual><geometry><cylinder radius="0.02" length="0.5"/></geometry><material name="silver"/></visual>
   </link>
-  <!-- 6. 센서 (위치 스위치 완료!) -->
+  <!-- 6. 기존 LiDAR 센서 -->
   <joint name="front_camera_joint" type="fixed">
     <parent link="front_mast_link"/><child link="front_camera"/>
@@ -95,4 +96,18 @@
     <origin xyz="0 0 0" rpy="0 0 0"/>
   </xacro:sensor_hokuyo>
+  <!-- 6a. Competition-compatible front downward RGB camera.
+       The initial mounting pose follows the 2026 Competition configuration.
+       Replace with measured robot geometry when available. -->
+  <xacro:sensor_rgb_camera
+      name="camera_front"
+      parent="base_link"
+      image_topic="camera_front/color/image_raw"
+      camera_info_topic="camera_front/color/camera_info"
+      width="424"
+      height="240"
+      update_rate="15"
+      hfov="1.50">
+    <origin xyz="0.42 0.0 1.48" rpy="0 1.2915 0"/>
+  </xacro:sensor_rgb_camera>
   <!-- 7. 메인 구동 바퀴 -->
   <joint name="left_wheel_hinge" type="continuous">

Commit message: Align simulated camera layout with Competition robot

File: orange_ros2/orange_description/xacro/orange_robot_simulation.xacro (robot description, xacro)
@@ -75,5 +75,5 @@
     <visual><geometry><cylinder radius="0.02" length="0.5"/></geometry><material name="silver"/></visual>
   </link>
-  <!-- 6. 기존 LiDAR 센서 -->
+  <!-- 6. Existing LiDAR sensors: intentionally unchanged for this checkpoint. -->
   <joint name="front_camera_joint" type="fixed">
     <parent link="front_mast_link"/><child link="front_camera"/>
@@ -96,9 +96,15 @@
     <origin xyz="0 0 0" rpy="0 0 0"/>
   </xacro:sensor_hokuyo>
-  <!-- 6a. Competition-compatible front downward RGB-D camera.
-       The color stream and mounting pose follow the validated 2026
-       Competition-style baseline. A co-located depth sensor shares the
-       same physical link and optical frame so the RGB contract remains
-       unchanged while depth can be validated independently. -->
+  <!--
+    6a. Competition camera layout.
+    The poses, stream roles, resolutions, and rates mirror the current
+    LCAS-Lab/TnTechIGVC2026 Competition branch:
+      * front RealSense D435I: downward RGB-D, 424x240 @ 15 Hz, 2.5 m depth clip
+      * rear RealSense D435I: downward RGB only, 424x240 @ 6 Hz
+      * ZED2: forward RGB-D, HD720 @ 15 Hz, 0.2--5.0 m depth
+    The RealSense topic names are kept compatible with the Competition lane
+    nodes. ZED topics match unified_lane_node's default subscriptions.
+  -->
+  <!-- Front downward RealSense-like RGB-D camera. -->
   <xacro:sensor_rgb_camera
       name="camera_front"
@@ -123,5 +129,51 @@
       hfov="1.50"
       near_clip="0.10"
-      far_clip="20.0"/>
+      far_clip="2.50"/>
+  <!-- Rear downward RealSense-like RGB camera; depth is disabled on Competition. -->
+  <xacro:sensor_rgb_camera
+      name="camera_rear"
+      parent="base_link"
+      image_topic="camera_rear/color/image_raw"
+      camera_info_topic="camera_rear/color/camera_info"
+      width="424"
+      height="240"
+      update_rate="6"
+      hfov="1.50">
+    <origin xyz="-0.42 0.0 1.0" rpy="0 1.2915 3.14159"/>
+  </xacro:sensor_rgb_camera>
+  <!--
+    ZED mount frame used by the real robot and NVBlox configuration.
+    The optical sensor is a zero-offset child so the public TF tree contains
+    both zed_camera_link and the ZED-style left optical frame.
+  -->
+  <link name="zed_camera_link"/>
+  <joint name="base_to_zed_camera" type="fixed">
+    <parent link="base_link"/>
+    <child link="zed_camera_link"/>
+    <origin xyz="0.43 0.0 1.58" rpy="0 0.43 0"/>
+  </joint>
+  <xacro:sensor_rgb_camera
+      name="zed_left_camera"
+      parent="zed_camera_link"
+      image_topic="zed/zed_node/rgb/image_rect_color"
+      camera_info_topic="zed/zed_node/rgb/camera_info"
+      width="1280"
+      height="720"
+      update_rate="15"
+      hfov="1.91986">
+    <origin xyz="0 0 0" rpy="0 0 0"/>
+  </xacro:sensor_rgb_camera>
+  <xacro:sensor_depth_camera
+      name="zed_depth"
+      parent="zed_left_camera_link"
+      image_topic="zed/zed_node/depth/depth_registered"
+      camera_info_topic="zed/zed_node/depth/camera_info"
+      frame_id="zed_left_camera_optical_frame"
+      width="1280"
+      height="720"
+      update_rate="15"
+      hfov="1.91986"
+      near_clip="0.20"
+      far_clip="5.0"/>
   <!-- 7. 메인 구동 바퀴 -->
   <joint name="left_wheel_hinge" type="continuous">
